Commit message: fix: 修正 IRB140 URDF visual origin 及 joint4 xyz

File: model/robot/IRB140/IRB140.urdf (robot description, URDF)
Before this commit: robot IRB140, 8 links, 7 joints
Joints:
- joint joint4: origin xyz=0 0 380 rpy=1.5708 0 0 -> xyz=0 -380 0 rpy=1.5708 0 0

Commit message: Unify robot, tool, and workpiece units around URDF scene
This change makes the runtime scene use a single length convention and documents why the conversions now happen in code instead of inside individual model files.

Why this was needed:

- We moved robot kinematics from hand-maintained DH/RBXML assumptions to an URDF + urdfdom + KDL pipeline.

- urdfdom/KDL require angular values in radians, but the project wants robot and tool URDF files to stay human-editable in degrees.

- Robot, tool, and workpiece assets were no longer using the same length convention after the URDF migration, which caused oversized tools/workpieces, oversized coordinate frames, and move/TCP editors applying mm values as if they were scene metres.

What this commit changes:

- Robot URDF files now author origin RPY values and angular limits in degrees, with explicit comments in the model files explaining that project convention.

- KdlChainBuilder now rewrites those robot URDF angle fields back to radians before handing XML to urdfdom/KDL, and only converts angular joint limits so prismatic limits are not accidentally rescaled in the future.

- RbXmlParser and test reference FK were updated to read the same robot URDF degree convention, so display code and regression checks stay aligned with runtime kinematics.

- Tool loading is now URDF-only. The old .tool/.xml compatibility files are removed, tool URDF RPY authoring is switched to degrees, and RobotController reads those degree values directly for display transforms.

- STEP workpieces are scaled from mm to the scene's metre-based runtime units at import time, and their tessellation deflection is adjusted so mesh quality stays equivalent to the previous 0.1 mm behaviour.

- MovementPanel, TCP pose editing, and coordinate trihedron sizes are updated so the UI still speaks mm/degrees to the operator while internal transforms remain in metres/degrees as expected by the current scene pipeline.

Result:

- Robot, tool, workpiece, and manipulation UI now agree on one runtime length unit.

- Human-authored URDF angle values remain readable in degrees.

- Future debugging is easier because the unit conversions now live in a few explicit places with comments instead of being hidden in asset data or accidental scale mismatches.

File: model/robot/IRB140/IRB140.urdf (robot description, URDF)
Before this commit: robot IRB140, 8 links, 7 joints
Joints:
- joint joint1: limit lower=-3.1416 upper=3.1416 effort=0 velocity=0 -> lower=-180 upper=180 effort=0 velocity=0
- joint joint2: limit lower=-1.5708 upper=1.9199 effort=0 velocity=0 -> lower=-90 upper=110 effort=0 velocity=0; origin xyz=70 0 0 rpy=-1.5708 0 0 -> xyz=70 0 0 rpy=-90 0 0
- joint joint3: limit lower=-4.0143 upper=0.8727 effort=0 velocity=0 -> lower=-230 upper=50 effort=0 velocity=0
- joint joint4: limit lower=-3.4907 upper=3.4907 effort=0 velocity=0 -> lower=-200 upper=200 effort=0 velocity=0; origin xyz=0 -380 0 rpy=1.5708 0 0 -> xyz=0 -380 0 rpy=90 0 0
- joint joint5: limit lower=-2.0071 upper=2.0071 effort=0 velocity=0 -> lower=-115 upper=115 effort=0 velocity=0; origin xyz=0 0 0 rpy=-1.5708 0 0 -> xyz=0 0 0 rpy=-90 0 0
- joint joint6: limit lower=-6.9813 upper=6.9813 effort=0 velocity=0 -> lower=-400 upper=400 effort=0 velocity=0; origin xyz=0 0 0 rpy=1.5708 0 0 -> xyz=0 0 0 rpy=90 0 0

File: model/robot/irb2400/irb2400.urdf (robot description, URDF)
Before this commit: robot abb_irb2400, 9 links, 8 joints
Joints:
- joint joint_1: limit lower=-3.1416 upper=3.1416 effort=0 velocity=2.618 -> lower=-180 upper=180 effort=0 velocity=150
- joint joint_2: limit lower=-1.7453 upper=1.9199 effort=0 velocity=2.618 -> lower=-100 upper=110 effort=0 velocity=150
- joint joint_3: limit lower=-1.0472 upper=1.1345 effort=0 velocity=2.618 -> lower=-60 upper=65 effort=0 velocity=150
- joint joint_4: limit lower=-3.49 upper=3.49 effort=0 velocity=6.2832 -> lower=-200 upper=200 effort=0 velocity=360
- joint joint_5: limit lower=-2.0944 upper=2.0944 effort=0 velocity=6.2832 -> lower=-120 upper=120 effort=0 velocity=360
- joint joint_6: limit lower=-6.9813 upper=6.9813 effort=0 velocity=7.854 -> lower=-400 upper=400 effort=0 velocity=450
- joint joint_6-tool0: origin xyz=0 0 0 rpy=0 1.57079632679 0 -> xyz=0 0 0 rpy=0 90 0
